File: PCB/Digital_Praytime_Display_P4.75_v0.9.brd (EAGLE design)
At the start: 90.9 x 58.8 mm, 54 parts, among them IC2 24C04SN, IC4 74HC245DW, IC5 74HC245DW, T1 BSS138, T3 BSS138, U1 STM32F103C8T6, X2 MSTBA2

Commit message: add some code and pcb
Parts:
- removed IC2: 24C04SN, microchip:SO-08
- removed J1, J2: (no value), rcl:R0402
- removed JP10: (no value), pinhead:1X01
- removed JP4, JP9: (no value), pinhead:1X05
- removed JP6: (no value), pinhead:2X04
- removed R13: 4K7, rcl:R0805
- removed R15, R16: 100, rcl:R0805
- removed R7, R9: 10K, rcl:R0805
- removed TP1, TP2, TP3: TPSQPAD1-13Y, testpad:P1-13Y
- added H4: MOUNT-HOLE3.0, holes:3,0
- added SJ2, SJ3, SJ4: (no value), jumper:SJ
- added X1: 057-016-1, con-panduit:057-016-1
- JP2: device pinhead:2X08 -> pinhead:1X06
- R11: value (none) -> 4K7
- R12: value (none) -> 100
- T2: device transistor:SOT23-BEC -> transistor:TO126V
- moved SJ1 38.4 mm to (17.9, 26.9), turned to 0 degrees
- moved T2 37.4 mm to (50.5, 45.7), flipped to the top, turned to 180 degrees
- moved R12 27.9 mm to (38.2, 36.7), turned to 0 degrees
- moved R11 24.6 mm to (45.5, 44.3), turned to 180 degrees
- moved JP2 20.7 mm to (44.3, 9.65), turned to 270 degrees
- moved JP5 13.1 mm to (67.3, 0.76)
- moved JP7 13.1 mm to (63.8, 0.76)
- moved G1 12.2 mm to (63.7, 12.5), turned to 0 degrees
- moved C3 8.02 mm to (13.8, 35.4), turned to 270 degrees
- moved C2 7.37 mm to (18.8, 44.8)
- moved C6 7.37 mm to (23.7, 44.8)
- moved JP8 7.37 mm to (18.8, 52.3)
- moved R1 7.37 mm to (15.0, 47.4)
- moved R4 7.37 mm to (19.6, 47.4)
- moved R6 7.37 mm to (24.0, 47.4)
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Connections:
- removed net CLK7: IC5.4, U1.3
- removed net CLK_SEG: IC5.16, JP4.4
- removed net DT7: IC5.2, U1.1
- removed net DT_SEG: IC5.18, JP4.2
- removed net GPS_ON: U1.29
- removed net N$10: JP6.4
- removed net N$123: IC2.7, SJ1.1
- removed net N$17: R13.1, R15.1, TP1.TP
- removed net N$18: R15.2, T2.C
- removed net N$19: JP6.5, R7.2
- removed net N$20: JP6.6
- removed net N$21: R16.2, T2.B
- removed net N$7: JP6.3, R9.2
- removed net N$8: J2.1, JP2.10
- removed net RST: R7.1, U1.37
- removed net RX3: JP6.1, U1.36
- removed net STR7: IC5.3, U1.2
- removed net STR_SEG: IC5.17, JP4.3
- removed net TX3: JP6.8, U1.35
- removed net WIFI: JP6.7, TP2.TP
- removed net WIFI_ON: R16.1, U1.34
- new net BL: JP3.5, T2.2
- new net BL_POW: R12.2, U1.29
- new net INT: JP2.5, U1.15
- new net N$12: SJ1.1, U1.8
- net +3V3: no longer R13.2, R9.1, TP3.TP
- net +5V: now also JP2.2, R11.2, T2.1; no longer JP3.5, JP4.1, JP9.1
- net 3V3: no longer IC2.8, R11.1, R12.1, SJ1.2
- net A: now also X1.2; no longer JP2.2
- net B: now also X1.4; no longer JP2.4
- net C: now also X1.6; no longer JP2.6
- net CLK: now also X1.16; no longer JP2.16
- net D: now also X1.8; no longer JP2.8
- net G1: now also SJ3.1; no longer J2.2
- net G1_BUFF: now also SJ2.2; no longer U1.9
- net G2: now also SJ4.1; no longer J1.2
- net G2_BUFF: now also SJ1.2; no longer U1.8
- net GND: now also X1.1, X1.3, X1.5; no longer IC2.4, JP2.3, JP2.5, JP4.5, JP6.2, JP9.5, T2.E
- net N$1: now also R11.1, R12.1, T2.3; no longer J1.1, JP2.12
- net N$13: now also SJ2.1, U1.9; no longer JP9.2
- net N$14: now also SJ4.2, X1.12; no longer JP9.3
- net N$15: now also SJ3.2, X1.10; no longer JP9.4
- net OE: now also X1.7; no longer JP2.7
- net R1: now also X1.9; no longer JP2.9
- net R2: now also X1.11; no longer JP2.11
- net RSV: no longer JP10.1
- net RSV_BUFF: no longer U1.15
- net SCL: now also JP2.4; no longer IC2.6, R12.2
- net SDA: now also JP2.3; no longer IC2.5, R11.2
- net STB: now also X1.14; no longer JP2.14
Routing:
- net 3V3: track 50.5 -> 0.00 mm, vias 2 -> 0
- net +3V3: track 107.6 -> 67.7 mm, vias 2 -> 0
- net GND: track 474.9 -> 441.9 mm
- net INT: track 0.00 -> 23.9 mm
- net CLK_SEG: track 20.1 -> 0.00 mm
- net STR_SEG: track 19.3 -> 0.00 mm
- net DT_SEG: track 18.3 -> 0.00 mm
- net RX3: track 18.1 -> 0.00 mm
- net TX3: track 17.6 -> 0.00 mm
- net +5V: track 174.6 -> 158.1 mm
- net N$7: track 12.6 -> 0.00 mm
- net N$17: track 12.2 -> 0.00 mm
- net DT7: track 12.0 -> 0.00 mm
- net N$1: track 5.33 -> 17.0 mm
- net STR7: track 10.4 -> 0.00 mm
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Other:
- board size 90.9 x 58.8 mm -> 88.4 x 58.8 mm
- board text added: "DPD_P4_7S_ver.0.9"
- board text removed: "DPD_P4_7S_ver.1.4"
