File: PCB/Digital_Praytime_Display_P4.75_v0.9.sch (EAGLE design)
At the start: 54 parts, among them IC2 24C04SN, IC4 74HC245DW, IC5 74HC245DW, T1 BSS138, T3 BSS138, U1 STM32F103C8T6, X2 MSTBA2

Commit message: add some code and pcb
Parts:
- removed IC2: 24C04SN, microchip:24C04SN
- removed J1, J2: (no value), rcl:R-EU_R0402
- removed JP10: (no value), pinhead:PINHD-1X1
- removed JP4, JP9: (no value), pinhead:PINHD-1X5
- removed JP6: (no value), pinhead:PINHD-2X4
- removed R13: 4K7, rcl:R-US_R0805
- removed R15, R16: 100, rcl:R-US_R0805
- removed R7, R9: 10K, rcl:R-US_R0805
- removed TP1, TP2, TP3: TPSQPAD1-13Y, testpad:TPSQPAD1-13Y
- added H4: MOUNT-HOLE3.0, holes:MOUNT-HOLE3.0
- added SJ2, SJ3, SJ4: (no value), jumper:SJ
- added X1: 057-016-1, con-panduit:057-016-1
- JP2: device pinhead:PINHD-2X8 -> pinhead:PINHD-1X6
- R11: value (none) -> 4K7
- R12: value (none) -> 100
- T2: device transistor:MMBT2222ALT1-NPN-SOT23-BEC -> transistor:-PNP-TO126V
Connections:
- removed net CLK7: IC5A.A3, U1.PB14
- removed net CLK_SEG: IC5A.B3, JP4.4
- removed net DT7: IC5A.A1, U1.PB12
- removed net DT_SEG: IC5A.B1, JP4.2
- removed net GPS_ON: U1.PA4
- removed net N$10: JP6.4
- removed net N$123: IC2.WP, SJ1.1
- removed net N$17: R13.1, R15.1, TP1.TP
- removed net N$18: R15.2, T2.C
- removed net N$19: JP6.5, R7.2
- removed net N$20: JP6.6
- removed net N$21: R16.2, T2.B
- removed net N$7: JP6.3, R9.2
- removed net N$8: J2.1, JP2.10
- removed net RST: R7.1, U1.RST
- removed net RX3: JP6.1, U1.PB11
- removed net STR7: IC5A.A2, U1.PB13
- removed net STR_SEG: IC5A.B2, JP4.3
- removed net TX3: JP6.8, U1.PB10
- removed net WIFI: JP6.7, TP2.TP
- removed net WIFI_ON: R16.1, U1.PB1
- new net BL: JP3.5, T2.C
- new net BL_POW: R12.2, U1.PA4
- new net INT: JP2.5, U1.PB7
- new net N$12: SJ1.1, U1.PA11
- net +3V3: no longer R13.2, R9.1, TP3.TP
- net +5V: now also JP2.2, R11.2, T2.E; no longer JP3.5, JP4.1, JP9.1
- net 3V3: no longer IC2.VCC, R11.1, R12.1, SJ1.2
- net A: now also X1-2.S; no longer JP2.2
- net B: now also X1-4.S; no longer JP2.4
- net C: now also X1-6.S; no longer JP2.6
- net CLK: now also X1-16.S; no longer JP2.16
- net D: now also X1-8.S; no longer JP2.8
- net G1: now also SJ3.1; no longer J2.2
- net G1_BUFF: now also SJ2.2; no longer U1.PA12
- net G2: now also SJ4.1; no longer J1.2
- net G2_BUFF: now also SJ1.2; no longer U1.PA11
- net GND: now also X1-1.S, X1-3.S, X1-5.S; no longer IC2.GND, JP2.3, JP2.5, JP4.5, JP6.2, JP9.5, T2.E
- net N$1: now also R11.1, R12.1, T2.B; no longer J1.1, JP2.12
- net N$13: now also SJ2.1, U1.PA12; no longer JP9.2
- net N$14: now also SJ4.2, X1-12.S; no longer JP9.3
- net N$15: now also SJ3.2, X1-10.S; no longer JP9.4
- net OE: now also X1-7.S; no longer JP2.7
- net R1: now also X1-9.S; no longer JP2.9
- net R2: now also X1-11.S; no longer JP2.11
- net RSV: no longer JP10.1
- net RSV_BUFF: no longer U1.PB7
- net SCL: now also JP2.4; no longer IC2.SCL, R12.2
- net SDA: now also JP2.3; no longer IC2.SDA, R11.2
- net STB: now also X1-14.S; no longer JP2.14
Other:
- moved on the sheet: R11, R12, SJ1
